File: hardware/sensor-test/kicad/hall-front-end.kicad_sch (KiCad schematic)
At the start: 15 parts, among them U4 TPS22919DCKR, U5 TMUX1208PWR, U6 DRV5055A3QDBZR, U7 DRV5055A3QDBZR, U8 DRV5055A3QDBZR, U9 DRV5055A3QDBZR

Commit message: Fix TMUX1208 NC pin placement
Connections:
- net HALL_5V: no longer U5.3 (NC)
- no-connect marks 5 -> 6
Changed lines of the file:
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@@
   (no_connect (at 117.3 92.3))
   (no_connect (at 117.3 89.76))
+  (no_connect (at 142.7 89.76))
 (label "VBUS" (at 36.11 50.08 0)
     (effects (font (size 1.27 1.27)) (justify left bottom))

Commit message: Add Hall rail input decoupling and measurement test pads
Parts:
- added C25: 1u, Capacitor_SMD:C_0603_1608Metric, symbol Device:C
- added TP1: VBUS, TestPoint:TestPoint_Pad_D1.5mm, symbol Connector:TestPoint
- added TP2: HALL_5V, TestPoint:TestPoint_Pad_D1.5mm, symbol Connector:TestPoint
- added TP3: H0_RAW, TestPoint:TestPoint_Pad_D1.5mm, symbol Connector:TestPoint
- added TP4: H1_RAW, TestPoint:TestPoint_Pad_D1.5mm, symbol Connector:TestPoint
- added TP5: H2_RAW, TestPoint:TestPoint_Pad_D1.5mm, symbol Connector:TestPoint
- added TP6: H3_RAW, TestPoint:TestPoint_Pad_D1.5mm, symbol Connector:TestPoint
- added TP7: MUX_D, TestPoint:TestPoint_Pad_D1.5mm, symbol Connector:TestPoint
- added TP8: ADC_SENSE, TestPoint:TestPoint_Pad_D1.5mm, symbol Connector:TestPoint
- added TP9: GND, TestPoint:TestPoint_Pad_D1.5mm, symbol Connector:TestPoint
Connections:
- net ADC_SENSE: now also TP8.1
- net GND: now also C25.1, TP9.1
- net HALL_5V: now also TP2.1
- net MUX_D: now also TP7.1
- net VBUS: now also C25.2, TP1.1
- net H0 renamed H0_RAW
- net H0_RAW: now also TP3.1
- net H1 renamed H1_RAW
- net H1_RAW: now also TP4.1
- net H2 renamed H2_RAW
- net H2_RAW: now also TP5.1
- net H3 renamed H3_RAW
- net H3_RAW: now also TP6.1
Changed lines of the file:
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@@
     (effects (font (size 1.27 1.27)) (justify left bottom))
   )
-  (label "H0" (at 117.3 117.7 0)
-    (effects (font (size 1.27 1.27)) (justify left bottom))
-  )
-  (label "H1" (at 117.3 112.62 0)
-    (effects (font (size 1.27 1.27)) (justify left bottom))
-  )
-  (label "H2" (at 117.3 107.54 0)
-    (effects (font (size 1.27 1.27)) (justify left bottom))
-  )
-  (label "H3" (at 117.3 102.46 0)
+  (label "H0_RAW" (at 117.3 117.7 0)
+    (effects (font (size 1.27 1.27)) (justify left bottom))
+  )
+  (label "H1_RAW" (at 117.3 112.62 0)
+    (effects (font (size 1.27 1.27)) (justify left bottom))
+  )
+  (label "H2_RAW" (at 117.3 107.54 0)
+    (effects (font (size 1.27 1.27)) (justify left bottom))
+  )
+  (label "H3_RAW" (at 117.3 102.46 0)
     (effects (font (size 1.27 1.27)) (justify left bottom))
   )
@@
     (effects (font (size 1.27 1.27)) (justify left bottom))
   )
-  (label "H0" (at 62.62 90 0)
+  (label "H0_RAW" (at 62.62 90 0)
     (effects (font (size 1.27 1.27)) (justify left bottom))
   )
@@
     (effects (font (size 1.27 1.27)) (justify left bottom))
   )
-  (label "H1" (at 62.62 118 0)
+  (label "H1_RAW" (at 62.62 118 0)
     (effects (font (size 1.27 1.27)) (justify left bottom))
   )
@@
     (effects (font (size 1.27 1.27)) (justify left bottom))
   )
-  (label "H2" (at 62.62 146 0)
+  (label "H2_RAW" (at 62.62 146 0)
     (effects (font (size 1.27 1.27)) (justify left bottom))
   )
@@
     (effects (font (size 1.27 1.27)) (justify left bottom))
   )
-  (label "H3" (at 62.62 174 0)
+  (label "H3_RAW" (at 62.62 174 0)
     (effects (font (size 1.27 1.27)) (justify left bottom))
   )
@@
     )
   )
+  (symbol (lib_id "Device:C") (at 72 45 0) (unit 1)
+    (in_bom yes) (on_board yes) (dnp no)
+    (property "Reference" "C25" (at 74.54 43.73 0) (effects (font (size 1.27 1.27)) (justify left)))
+    (property "Value" "1u" (at 74.54 46.27 0) (effects (font (size 1.27 1.27)) (justify left)))
+    (property "Footprint" "Capacitor_SMD:C_0603_1608Metric" (at 72.9652 41.19 0) (effects (font (size 1.27 1.27)) hide))
+    (property "Datasheet" "~" (at 72 45 0) (effects (font (size 1.27 1.27)) hide))
+    (property "LCSC" "" (at 72 45 0) (effects (font (size 1.27 1.27)) hide))
+    (pin "1")
+    (pin "2")
+    (instances
+      (project "hall-front-end"
+        (path "/a1000000-0000-0000-0000-000000000001"
+          (reference "C25") (unit 1)
+        )
+      )
+    )
+  )
+  (label "VBUS" (at 72 48.81 0)
+    (effects (font (size 1.27 1.27)) (justify left bottom))
+  )
+  (label "GND" (at 72 41.19 0)
+    (effects (font (size 1.27 1.27)) (justify left bottom))
+  )
+  (symbol (lib_id "Connector:TestPoint") (at 235 40 0) (unit 1)
+    (in_bom no) (on_board yes) (dnp no)
+    (property "Reference" "TP1" (at 235 33.65 0) (effects (font (size 1.27 1.27))))
+    (property "Value" "VBUS" (at 237.54 35.428 0) (effects (font (size 1.27 1.27)) (justify left)))
+    (property "Footprint" "TestPoint:TestPoint_Pad_D1.5mm" (at 240.08 40 0) (effects (font (size 1.27 1.27)) hide))
+    (property "Datasheet" "~" (at 240.08 40 0) (effects (font (size 1.27 1.27)) hide))
+    (pin "1")
+    (instances
+      (project "hall-front-end"
+        (path "/a1000000-0000-0000-0000-000000000001"
+          (reference "TP1") (unit 1)
+        )
+      )
+    )
+  )
+  (label "VBUS" (at 235 40 0)
+    (effects (font (size 1.27 1.27)) (justify left bottom))
+  )
+  (symbol (lib_id "Connector:TestPoint") (at 235 52 0) (unit 1)
+    (in_bom no) (on_board yes) (dnp no)
+    (property "Reference" "TP2" (at 235 45.65 0) (effects (font (size 1.27 1.27))))
+    (property "Value" "HALL_5V" (at 237.54 47.428 0) (effects (font (size 1.27 1.27)) (justify left)))
+    (property "Footprint" "TestPoint:TestPoint_Pad_D1.5mm" (at 240.08 52 0) (effects (font (size 1.27 1.27)) hide))
+    (property "Datasheet" "~" (at 240.08 52 0) (effects (font (size 1.27 1.27)) hide))
+    (pin "1")
+    (instances
+      (project "hall-front-end"
+        (path "/a1000000-0000-0000-0000-000000000001"
+          (reference "TP2") (unit 1)
+        )
+      )
+    )
+  )
+  (label "HALL_5V" (at 235 52 0)
+    (effects (font (size 1.27 1.27)) (justify left bottom))
+  )
+  (symbol (lib_id "Connector:TestPoint") (at 235 68 0) (unit 1)
+    (in_bom no) (on_board yes) (dnp no)
+    (property "Reference" "TP3" (at 235 61.65 0) (effects (font (size 1.27 1.27))))
+    (property "Value" "H0_RAW" (at 237.54 63.428 0) (effects (font (size 1.27 1.27)) (justify left)))
+    (property "Footprint" "TestPoint:TestPoint_Pad_D1.5mm" (at 240.08 68 0) (effects (font (size 1.27 1.27)) hide))
+    (property "Datasheet" "~" (at 240.08 68 0) (effects (font (size 1.27 1.27)) hide))
+    (pin "1")
+    (instances
+      (project "hall-front-end"
+        (path "/a1000000-0000-0000-0000-000000000001"
+          (reference "TP3") (unit 1)
+        )
+      )
+    )
+  )
+  (label "H0_RAW" (at 235 68 0)
+    (effects (font (size 1.27 1.27)) (justify left bottom))
+  )
+  (symbol (lib_id "Connector:TestPoint") (at 235 80 0) (unit 1)
+    (in_bom no) (on_board yes) (dnp no)
+    (property "Reference" "TP4" (at 235 73.65 0) (effects (font (size 1.27 1.27))))
+    (property "Value" "H1_RAW" (at 237.54 75.428 0) (effects (font (size 1.27 1.27)) (justify left)))
+    (property "Footprint" "TestPoint:TestPoint_Pad_D1.5mm" (at 240.08 80 0) (effects (font (size 1.27 1.27)) hide))
+    (property "Datasheet" "~" (at 240.08 80 0) (effects (font (size 1.27 1.27)) hide))
+    (pin "1")
+    (instances
+      (project "hall-front-end"
+        (path "/a1000000-0000-0000-0000-000000000001"
+          (reference "TP4") (unit 1)
+        )
+      )
+    )
+  )
+  (label "H1_RAW" (at 235 80 0)
+    (effects (font (size 1.27 1.27)) (justify left bottom))
+  )
+  (symbol (lib_id "Connector:TestPoint") (at 235 92 0) (unit 1)
+    (in_bom no) (on_board yes) (dnp no)
+    (property "Reference" "TP5" (at 235 85.65 0) (effects (font (size 1.27 1.27))))
+    (property "Value" "H2_RAW" (at 237.54 87.428 0) (effects (font (size 1.27 1.27)) (justify left)))
+    (property "Footprint" "TestPoint:TestPoint_Pad_D1.5mm" (at 240.08 92 0) (effects (font (size 1.27 1.27)) hide))
+    (property "Datasheet" "~" (at 240.08 92 0) (effects (font (size 1.27 1.27)) hide))
+    (pin "1")
+    (instances
+      (project "hall-front-end"
+        (path "/a1000000-0000-0000-0000-000000000001"
+          (reference "TP5") (unit 1)
+        )
+      )
+    )
+  )
+  (label "H2_RAW" (at 235 92 0)
+    (effects (font (size 1.27 1.27)) (justify left bottom))
+  )
+  (symbol (lib_id "Connector:TestPoint") (at 235 104 0) (unit 1)
+    (in_bom no) (on_board yes) (dnp no)
+    (property "Reference" "TP6" (at 235 97.65 0) (effects (font (size 1.27 1.27))))
+    (property "Value" "H3_RAW" (at 237.54 99.428 0) (effects (font (size 1.27 1.27)) (justify left)))
+    (property "Footprint" "TestPoint:TestPoint_Pad_D1.5mm" (at 240.08 104 0) (effects (font (size 1.27 1.27)) hide))
+    (property "Datasheet" "~" (at 240.08 104 0) (effects (font (size 1.27 1.27)) hide))
+    (pin "1")
+    (instances
+      (project "hall-front-end"
+        (path "/a1000000-0000-0000-0000-000000000001"
+          (reference "TP6") (unit 1)
+        )
+      )
+    )
+  )
+  (label "H3_RAW" (at 235 104 0)
+    (effects (font (size 1.27 1.27)) (justify left bottom))
+  )
+  (symbol (lib_id "Connector:TestPoint") (at 235 120 0) (unit 1)
+    (in_bom no) (on_board yes) (dnp no)
+    (property "Reference" "TP7" (at 235 113.65 0) (effects (font (size 1.27 1.27))))
+    (property "Value" "MUX_D" (at 237.54 115.428 0) (effects (font (size 1.27 1.27)) (justify left)))
+    (property "Footprint" "TestPoint:TestPoint_Pad_D1.5mm" (at 240.08 120 0) (effects (font (size 1.27 1.27)) hide))
+    (property "Datasheet" "~" (at 240.08 120 0) (effects (font (size 1.27 1.27)) hide))
+    (pin "1")
+    (instances
+      (project "hall-front-end"
+        (path "/a1000000-0000-0000-0000-000000000001"
+          (reference "TP7") (unit 1)
+        )
+      )
+    )
+  )
+  (label "MUX_D" (at 235 120 0)
+    (effects (font (size 1.27 1.27)) (justify left bottom))
+  )
+  (symbol (lib_id "Connector:TestPoint") (at 235 132 0) (unit 1)
+    (in_bom no) (on_board yes) (dnp no)
+    (property "Reference" "TP8" (at 235 125.65 0) (effects (font (size 1.27 1.27))))
+    (property "Value" "ADC_SENSE" (at 237.54 127.428 0) (effects (font (size 1.27 1.27)) (justify left)))
+    (property "Footprint" "TestPoint:TestPoint_Pad_D1.5mm" (at 240.08 132 0) (effects (font (size 1.27 1.27)) hide))
+    (property "Datasheet" "~" (at 240.08 132 0) (effects (font (size 1.27 1.27)) hide))
+    (pin "1")
+    (instances
+      (project "hall-front-end"
+        (path "/a1000000-0000-0000-0000-000000000001"
+          (reference "TP8") (unit 1)
+        )
+      )
+    )
+  )
+  (label "ADC_SENSE" (at 235 132 0)
+    (effects (font (size 1.27 1.27)) (justify left bottom))
+  )
+  (symbol (lib_id "Connector:TestPoint") (at 235 148 0) (unit 1)
+    (in_bom no) (on_board yes) (dnp no)
+    (property "Reference" "TP9" (at 235 141.65 0) (effects (font (size 1.27 1.27))))
+    (property "Value" "GND" (at 237.54 143.428 0) (effects (font (size 1.27 1.27)) (justify left)))
+    (property "Footprint" "TestPoint:TestPoint_Pad_D1.5mm" (at 240.08 148 0) (effects (font (size 1.27 1.27)) hide))
+    (property "Datasheet" "~" (at 240.08 148 0) (effects (font (size 1.27 1.27)) hide))
+    (pin "1")
+    (instances
+      (project "hall-front-end"
+        (path "/a1000000-0000-0000-0000-000000000001"
+          (reference "TP9") (unit 1)
+        )
+      )
+    )
+  )
+  (label "GND" (at 235 148 0)
+    (effects (font (size 1.27 1.27)) (justify left bottom))
+  )
   (sheet_instances

Commit message: Expose unused TMUX channels on evaluation test pads
Parts:
- added TP10: MUX_S5_SPARE, TestPoint:TestPoint_Pad_D1.5mm, symbol Connector:TestPoint
- added TP11: MUX_S6_SPARE, TestPoint:TestPoint_Pad_D1.5mm, symbol Connector:TestPoint
- added TP12: MUX_S7_SPARE, TestPoint:TestPoint_Pad_D1.5mm, symbol Connector:TestPoint
- added TP13: MUX_S8_SPARE, TestPoint:TestPoint_Pad_D1.5mm, symbol Connector:TestPoint
Connections:
- net MUX_S7_SPARE: now reaches U5.4 (S1)
- net MUX_S7_SPARE: now also TP12.1
- net MUX_S5_SPARE: now reaches U5.5 (S2)
- net MUX_S5_SPARE: now also TP10.1
- new net MUX_S6_SPARE: TP11.1
- new net MUX_S8_SPARE: TP13.1
- no-connect marks 6 -> 2
Changed lines of the file:
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@@
   )
 (no_connect (at 53.89 39.92))
-  (no_connect (at 117.3 97.38))
-  (no_connect (at 117.3 94.84))
-  (no_connect (at 117.3 92.3))
-  (no_connect (at 117.3 89.76))
   (no_connect (at 142.7 89.76))
 (label "VBUS" (at 36.11 50.08 0)
@@
     (effects (font (size 1.27 1.27)) (justify left bottom))
   )
+  (label "MUX_S5_SPARE" (at 117.3 97.38 0)
+    (effects (font (size 1.27 1.27)) (justify left bottom))
+  )
+  (label "MUX_S6_SPARE" (at 117.3 94.84 0)
+    (effects (font (size 1.27 1.27)) (justify left bottom))
+  )
+  (label "MUX_S7_SPARE" (at 117.3 92.3 0)
+    (effects (font (size 1.27 1.27)) (justify left bottom))
+  )
+  (label "MUX_S8_SPARE" (at 117.3 89.76 0)
+    (effects (font (size 1.27 1.27)) (justify left bottom))
+  )
+  (symbol (lib_id "Connector:TestPoint") (at 260 68 0) (unit 1)
+    (in_bom no) (on_board yes) (dnp no)
+    (property "Reference" "TP10" (at 260 61.65 0) (effects (font (size 1.27 1.27))))
+    (property "Value" "MUX_S5_SPARE" (at 262.54 63.428 0) (effects (font (size 1.27 1.27)) (justify left)))
+    (property "Footprint" "TestPoint:TestPoint_Pad_D1.5mm" (at 265.08 68 0) (effects (font (size 1.27 1.27)) hide))
+    (property "Datasheet" "~" (at 265.08 68 0) (effects (font (size 1.27 1.27)) hide))
+    (pin "1")
+    (instances
+      (project "hall-front-end"
+        (path "/a1000000-0000-0000-0000-000000000001"
+          (reference "TP10") (unit 1)
+        )
+      )
+    )
+  )
+  (label "MUX_S5_SPARE" (at 260 68 0)
+    (effects (font (size 1.27 1.27)) (justify left bottom))
+  )
+  (symbol (lib_id "Connector:TestPoint") (at 260 80 0) (unit 1)
+    (in_bom no) (on_board yes) (dnp no)
+    (property "Reference" "TP11" (at 260 73.65 0) (effects (font (size 1.27 1.27))))
+    (property "Value" "MUX_S6_SPARE" (at 262.54 75.428 0) (effects (font (size 1.27 1.27)) (justify left)))
+    (property "Footprint" "TestPoint:TestPoint_Pad_D1.5mm" (at 265.08 80 0) (effects (font (size 1.27 1.27)) hide))
+    (property "Datasheet" "~" (at 265.08 80 0) (effects (font (size 1.27 1.27)) hide))
+    (pin "1")
+    (instances
+      (project "hall-front-end"
+        (path "/a1000000-0000-0000-0000-000000000001"
+          (reference "TP11") (unit 1)
+        )
+      )
+    )
+  )
+  (label "MUX_S6_SPARE" (at 260 80 0)
+    (effects (font (size 1.27 1.27)) (justify left bottom))
+  )
+  (symbol (lib_id "Connector:TestPoint") (at 260 92 0) (unit 1)
+    (in_bom no) (on_board yes) (dnp no)
+    (property "Reference" "TP12" (at 260 85.65 0) (effects (font (size 1.27 1.27))))
+    (property "Value" "MUX_S7_SPARE" (at 262.54 87.428 0) (effects (font (size 1.27 1.27)) (justify left)))
+    (property "Footprint" "TestPoint:TestPoint_Pad_D1.5mm" (at 265.08 92 0) (effects (font (size 1.27 1.27)) hide))
+    (property "Datasheet" "~" (at 265.08 92 0) (effects (font (size 1.27 1.27)) hide))
+    (pin "1")
+    (instances
+      (project "hall-front-end"
+        (path "/a1000000-0000-0000-0000-000000000001"
+          (reference "TP12") (unit 1)
+        )
+      )
+    )
+  )
+  (label "MUX_S7_SPARE" (at 260 92 0)
+    (effects (font (size 1.27 1.27)) (justify left bottom))
+  )
+  (symbol (lib_id "Connector:TestPoint") (at 260 104 0) (unit 1)
+    (in_bom no) (on_board yes) (dnp no)
+    (property "Reference" "TP13" (at 260 97.65 0) (effects (font (size 1.27 1.27))))
+    (property "Value" "MUX_S8_SPARE" (at 262.54 99.428 0) (effects (font (size 1.27 1.27)) (justify left)))
+    (property "Footprint" "TestPoint:TestPoint_Pad_D1.5mm" (at 265.08 104 0) (effects (font (size 1.27 1.27)) hide))
+    (property "Datasheet" "~" (at 265.08 104 0) (effects (font (size 1.27 1.27)) hide))
+    (pin "1")
+    (instances
+      (project "hall-front-end"
+        (path "/a1000000-0000-0000-0000-000000000001"
+          (reference "TP13") (unit 1)
+        )
+      )
+    )
+  )
+  (label "MUX_S8_SPARE" (at 260 104 0)
+    (effects (font (size 1.27 1.27)) (justify left bottom))
+  )
